File: stm32mpu/stm32mpu/RAM.sch (KiCad schematic (older format))
At the start: 2 parts

Commit message: pre-leaving newfoundland
added a lot of stuff - unsure of what has changed
Parts:
- added C? (x15): 100nF, Capacitor_SMD:C_0402_1005Metric, symbol Device:C_Small
- added C? (x2): 10uF, Capacitor_SMD:C_0402_1005Metric, symbol Device:C_Small
- added C? (x12): 100n, Capacitor_SMD:C_0402_1005Metric, symbol Device:C_Small
- added C? (x2): 22uF, Capacitor_SMD:C_0402_1005Metric, symbol Device:C_Small
- added R? (x22): 56, Resistor_SMD:R_0402_1005Metric, symbol Device:R_Small
- added R?: 100, Resistor_SMD:R_0402_1005Metric, symbol Device:R_Small
- added R? (x2): 240, Resistor_SMD:R_0402_1005Metric, symbol Device:R_Small
- added R? (x2): 10k, symbol Device:R_Small
- added U? (x3): VREF_DDR, symbol mpu_symbols:VREF_DDR
- added U? (x5): VDD_DDR, symbol mpu_symbols:VDD_DDR
- added U?: VTT_DDR, symbol mpu_symbols:VTT_DDR
- U?: footprint BGA96C80P9X16_1400X800X120N -> stm32mpu_footprints:BGA96C80P9X16_1400X800X120N; Digikey (none) -> ‎557-2010-1-ND‎
- U?: symbol mpu_symbols:STM32MP157AAA3T -> stm32mpu-rescue:STM32MP157AAA3T-mpu_symbols
Connections:
- net +1V1: now reaches U?.A1 (VDDQ)
- net +1V1: now also U?.A8 (VDDQ), U?.AB19 (DDR_VREF), U?.B2 (VDD), U?.C1 (VDDQ), U?.C9 (VDDQ), U?.D2 (VDDQ), U?.D9 (VDD), U?.E9 (VDDQ), U?.F1 (VDDQ), U?.G7 (VDD), U?.H1 (VREFDQ), U?.H2 (VDDQ), U?.H9 (VDDQ), U?.K2 (VDD), U?.K8 (VDD), U?.M8 (VREFCA), U?.N1 (VDD), U?.N9 (VDD), U?.R1 (VDD), U?.R9 (VDD), C?.1, C?.1, C?.1, C?.1, C?.1, C?.1, C?.1, C?.1, C?.1, C?.1, C?.1, C?.1, C?.1, C?.1, C?.1, C?.1, C?.1, C?.1, C?.1, C?.1, C?.1, C?.1, C?.1, C?.1, C?.1, C?.1, C?.1, C?.1, C?.1, C?.1, C?.1, R?.1, R?.1, R?.1, R?.1, R?.1, R?.1, R?.1, R?.1, R?.1, R?.1, R?.1, R?.1, R?.1, R?.1, R?.1, R?.1, R?.1, R?.1, R?.1, R?.1, R?.1, R?.1, U?.1 (+1V1), U?.1 (+1V1), U?.1 (+1V1), U?.1 (+1V1), U?.1 (+1V1), U?.1 (+1V1), U?.1 (+1V1), U?.1 (+1V1), U?.1 (+1V1)
- net DDR0_DQ13: now reaches U?.A2 (DQ13)
- net DDR0_DQ13: now also U?.R20 (DDR_DQ13)
- net DDR0_DQ15: now reaches U?.A3 (DQ15)
- net DDR0_DQ15: now also U?.V21 (DDR_DQ15)
- net DDR0_DQ12: now reaches U?.A7 (DQ12)
- net DDR0_DQ12: now also U?.V20 (DDR_DQ12)
- net GND: now reaches U?.A9 (VSS)
- net GND: now also U?.B1 (VSSQ), U?.B3 (VSS), U?.B9 (VSSQ), U?.D1 (VSSQ), U?.D8 (VSSQ), U?.E1 (VSS), U?.E2 (VSSQ), U?.E8 (VSSQ), U?.F9 (VSSQ), U?.G1 (VSSQ), U?.G8 (VSS), U?.G9 (VSSQ), U?.J2 (VSS), U?.J8 (VSS), U?.M1 (VSS), U?.M9 (VSS), U?.P1 (VSS), U?.P9 (VSS), U?.T1 (VSS), U?.T9 (VSS), C?.2, C?.2, C?.2, C?.2, C?.2, C?.2, C?.2, C?.2, C?.2, C?.2, C?.2, C?.2, C?.2, C?.2, C?.2, C?.2, C?.2, C?.2, C?.2, C?.2, C?.2, C?.2, C?.2, C?.2, C?.2, C?.2, C?.2, C?.2, C?.2, C?.2, C?.2, R?.1, R?.1, R?.1, R?.1
- net DDR0_DQS1_N: now reaches U?.B7 (UDQS#)
- net DDR0_DQS1_N: now also U?.R22 (DDR_DQS1N)
- net DDR0_DQ14: now reaches U?.B8 (DQ14)
- net DDR0_DQ14: now also U?.U21 (DDR_DQ14)
- net DDR0_DQ11: now reaches U?.C2 (DQ11)
- net DDR0_DQ11: now also U?.T20 (DDR_DQ11)
- net DDR0_DQ9: now reaches U?.C3 (DQ9)
- net DDR0_DQ9: now also U?.R21 (DDR_DQ9)
- net DDR0_DQS1_P: now reaches U?.C7 (UDQS)
- net DDR0_DQS1_P: now also U?.T22 (DDR_DQS1P)
- net DDR0_DQ10: now reaches U?.C8 (DQ10)
- net DDR0_DQ10: now also U?.P21 (DDR_DQ10)
- net DDR0_UDM: now reaches U?.D3 (UDM)
- net DDR0_UDM: now also U?.G20 (DDR_DQM0)
- net DDR0_DQ8: now reaches U?.D7 (DQ8)
- net DDR0_DQ8: now also U?.N22 (DDR_DQ8)
- net DDR0_DQ0: now reaches U?.E3 (DQ0)
- net DDR0_DQ0: now also U?.E21 (DDR_DQ0)
- net DDR0_LDM: now reaches U?.E7 (LDM)
- net DDR0_LDM: now also U?.T21 (DDR_DQM1)
- net DDR0_DQ2: now reaches U?.F2 (DQ2)
- net DDR0_DQ2: now also U?.H21 (DDR_DQ2)
- net DDR0_DQS0_P: now reaches U?.F3 (LDQS)
- net DDR0_DQS0_P: now also U?.G22 (DDR_DQS0P)
- net DDR0_DQ1: now reaches U?.F7 (DQ1)
- net DDR0_DQ1: now also U?.F21 (DDR_DQ1)
- net DDR0_DQ3: now reaches U?.F8 (DQ3)
- net DDR0_DQ3: now also U?.E20 (DDR_DQ3)
- net DDR0_DQ6: now reaches U?.G2 (DQ6)
- net DDR0_DQ6: now also U?.H22 (DDR_DQ6)
- net DDR0_DQS0_N: now reaches U?.G3 (LDQS#)
- net DDR0_DQS0_N: now also U?.G21 (DDR_DQS0N)
- net DDR0_DQ4: now reaches U?.H3 (DQ4)
- net DDR0_DQ4: now also U?.J21 (DDR_DQ4)
- net DDR0_DQ7: now reaches U?.H7 (DQ7)
- net DDR0_DQ7: now also U?.G19 (DDR_DQ7)
- net DDR0_DQ5: now reaches U?.H8 (DQ5)
- net DDR0_DQ5: now also U?.H20 (DDR_DQ5)
- net DDR_RASN: now reaches U?.J3 (RAS#)
- net DDR_RASN: now also U?.M20 (DDR_RASN), R?.2
- net DDR_CLK_P: now reaches U?.J7 (CK)
- net DDR_CLK_P: now also U?.N21 (DDR_CLKN), R?.2
- net DDR_ODT: now reaches U?.K1 (ODT)
- net DDR_ODT: now also U?.L21 (DDR_ODT), R?.2
- net DDR_CASN: now reaches U?.K3 (CAS#)
- net DDR_CASN: now also U?.M22 (DDR_CASN), R?.2
- net DDR_CLK_N: now reaches U?.K7 (CK#)
- net DDR_CLK_N: now also U?.N20 (DDR_CLKP), R?.1
- net DDR_CKE: now reaches U?.K9 (CKE)
- net DDR_CKE: now also U?.R19 (DDR_CKE), R?.2, R?.2
- net DDR_CSN: now reaches U?.L2 (CS#)
- net DDR_CSN: now also U?.L18 (DDR_CSN), R?.2
- net DDR_WEN: now reaches U?.L3 (WE#)
- net DDR_WEN: now also U?.M21 (DDR_WEN), R?.2
- net DDR0_A10: now reaches U?.L7 (A10/AP)
- net DDR0_A10: now also U?.N18 (DDR_A10), R?.2
- net at U?.L8 (ZQ): now also R?.2
- net DDR0_BA0: now reaches U?.M2 (BA0)
- net DDR0_BA0: now also U?.K20 (DDR_BA0), R?.2
- net DDR0_BA2: now reaches U?.M3 (BA2)
- net DDR0_BA2: now also U?.K18 (DDR_BA2), R?.2
- net DDR0_A3: now reaches U?.N2 (A3)
- net DDR0_A3: now also U?.J19 (DDR_A3), R?.2
- net DDR0_A0: now reaches U?.N3 (A0)
- net DDR0_A0: now also U?.K19 (DDR_A0), R?.2
- net DDR0_A12: now reaches U?.N7 (A12/BC#)
- net DDR0_A12: now also U?.N19 (DDR_A12), R?.2
- net DDR0_BA1: now reaches U?.N8 (BA1)
- net DDR0_BA1: now also U?.R18 (DDR_BA1), R?.2
- net DDR0_A5: now reaches U?.P2 (A5)
- net DDR0_A5: now also U?.H19 (DDR_A5), R?.2
- net DDR0_A2: now reaches U?.P3 (A2)
- net DDR0_A2: now also U?.J18 (DDR_A2), R?.2
- net DDR0_A1: now reaches U?.P7 (A1)
- net DDR0_A1: now also U?.M18 (DDR_A1), R?.2
- net DDR0_A4: now reaches U?.P8 (A4)
- net DDR0_A4: now also U?.T18 (DDR_A4), R?.2
- net DDR0_A7: now reaches U?.R2 (A7)
- net DDR0_A7: now also U?.F18 (DDR_A7), R?.2
- net DDR0_A9: now reaches U?.R3 (A9)
- net DDR0_A9: now also U?.H18 (DDR_A9), R?.2
- net DDR0_A11: now reaches U?.R7 (A11)
- net DDR0_A11: now also U?.P19 (DDR_A11), R?.2
- net DDR0_A6: now reaches U?.R8 (A6)
- net DDR0_A6: now also U?.U19 (DDR_A6), R?.2
- net DDR0_RESET_N: now reaches U?.T2 (RESET#)
- net DDR0_RESET_N: now also U?.F19 (DDR_RESETN), R?.2
- net DDR0_A8: now reaches U?.T8 (A8)
- net DDR0_A8: now also U?.U18 (DDR_A8), R?.2
- net at U?.K22 (DDR_ZQ): now also R?.2
- no-connect marks 0 -> 28
Other:
- note added: "NOTE: 100ohm differential"
- note added: "NOTE: ODT for data, strobe and mask signals"
- note added: "NOTE: need to add decoupling for termination resistors"
- note added: "Place 10nF caps as close as possible to \nDDR_VREF pins on DRAM IC."
- note added: "Place 10nF caps as close as possible to power pins. \n10uF capacitors just need to be in near vicinity."
- moved on the sheet: U?, U?D
