File: stm32mpu/stm32mpu/power.sch (KiCad schematic (older format))
At the start: 27 parts

Commit message: pre-leaving newfoundland
added a lot of stuff - unsure of what has changed
Parts:
- removed C? (x3): C_Small, symbol Device:C_Small
- removed C? (x3): ???uF, symbol Device:C_Small
- removed L? (x3): ??? uH, symbol Device:L_Small
- removed R? (x2): ???, symbol Device:R_Small
- removed U? (x2): STM32MP157AAA3T, LFBGA448_18X18, symbol mpu_symbols:STM32MP157AAA3T
- added C?: ???uF, symbol Device:C_Small
- added C? (x3): 22uF, Capacitor_SMD:C_1206_3216Metric, symbol Device:C_Small
- added C?: 10uF, symbol Device:C_Small
- added C? (x3): 10uF, Capacitor_SMD:C_1206_3216Metric, symbol Device:C_Small
- added C?: 4.7uF, symbol Device:C_Small
- added J?: PWR_HEADER, symbol Connector_Generic:Conn_01x02
- added L? (x3): 1uH, Inductor_SMD:L_1008_2520Metric_Pad1.43x2.20mm_HandSolder, symbol Device:L_Small
- added R? (x6): 0, symbol Device:R_Small
- added U?: VREF_DDR, symbol mpu_symbols:VREF_DDR
- added U?: VTT_DDR, symbol mpu_symbols:VTT_DDR
- added U? (x3): VDD, symbol mpu_symbols:VDD
- added U?: VDD_CORE, symbol mpu_symbols:VDD_CORE
- added U? (x2): VDD_DDR, symbol mpu_symbols:VDD_DDR
- C?: value ???uF -> 22uF; footprint (none) -> Capacitor_SMD:C_1206_3216Metric; Digikey (none) -> 399-4937-1-ND
- C?: value ???uF -> 10uF; footprint (none) -> Capacitor_SMD:C_1206_3216Metric; Digikey (none) -> 399-4937-1-ND
- C? (x2): value ???uF -> 4.7uF
- C? (x3): value ???uF -> 1uF
- C? (x2): value ???uF -> 10uF
- C?: value ???nF -> 10nF
- L?: value ??? uH -> 1uH; footprint (none) -> Inductor_SMD:L_1008_2520Metric_Pad1.43x2.20mm_HandSolder; Digikey (none) -> SRP2512A-1R0MCT-ND
- U?: value STPMIC1APQR -> STPMIC1DPQR; symbol mpu_symbols:STPMIC1APQR -> stm32mpu-rescue:STPMIC1APQR-mpu_symbols
Connections:
- net VDD_CORE is gone; now on net +1V1: C?.1, L?.2, U?.5 (VOUT1)
- net VREF_DDR is gone; now on net +1V1: C?.1, U?.16 (VREFDDR)
- net VTT_DDR is gone; now on net +1V1: C?.1, U?.14 (LDO3OUT)
- net GND: now also C?.2, C?.2, C?.2, C?.2, C?.2, C?.2, C?.2, C?.2, C?.2, J?.2 (Pin_2)
- net at U?.18 (LDO2OUT): now also R?.2
- net at U?.21 (LDO6OUT): now also R?.2
- net at U?.23 (LDO1OUT): now also R?.2
- net +1V2: now reaches U?.27 (VOUT4)
- net +1V2: now also C?.1, L?.2
- net +1V1: now reaches U?.31 (VOUT3)
- net +1V1: now also C?.1, C?.1, R?.2, U?.13 (LDO3IN), U?.22 (LDO16IN), U?.9 (VOUT2), C?.1, C?.1, L?.2, L?.2, U?.1 (+1V1), U?.1 (+1V1), U?.1 (+1V1), U?.1 (+1V1), U?.1 (+1V1), U?.1 (+1V1), U?.1 (+1V1), U?.1 (+1V1)
- net at U?.39 (LDO4OUT): now also R?.2
- net at U?.40 (INTLDO): now also C?.1
- net at R?.1, U?.42 (VIO): now also C?.1
- net 1V2: no longer names the net of U?.25 (VLX4)
- net 1V2: now also L?.1
- net STPMIC1_INTn renamed STMPIC_INTn
- net STPMIC1_PWRCTRL renamed STPMIC_PWRCTRL
- net STPMIC1_RSTn renamed STMPIC_RSTn
- net STPMIC1_WAKEUP renamed STMPIC_WAKEUP
- removed net VDD: C?.1, R?.2, U?.22 (LDO16IN), U?.29 (VLX3)
- net VDDA: no longer names the net of U?.20 (LDO5OUT)
- net VDDA: now also R?.2; no longer C?.1
- removed net VDD_DDR: C?.1, U?.11 (VLX2), U?.13 (LDO3IN)
- net VIN: no longer names the net of C?.1, C?.1, C?.1, U?.12 (BUCK2IN), U?.19 (LDO25IN), U?.28 (BUCK3IN), U?.36 (VIN), U?.8 (BUCK1IN)
- net VIN: now also C?.1, C?.1, C?.1, J?.1 (Pin_1), R?.2; no longer U?.24 (BUCK4IN)
- new net: L?.1, U?.11 (VLX2)
- new net: C?.1, R?.1, U?.24 (BUCK4IN)
- new net: L?.1, U?.29 (VLX3)
- new net +3V3: C?.1, R?.1
- no-connect marks 9 -> 10
Other:
- note added: "LDO5OUT is 350mA\nSD Card Current: 100mA\nEth Phy Current: 83mA\nBUT IT HAS TO BE PROGRAMMED"
- note added: "MPU \nDECOUPLING"
- note added: "Note: LDOs pinned out in case they are needed."
- note added: "VDD_CORE = BUCK1 = 1V2 (cont. 1500mA) (Ind. Peak 2A)\nVDD_DDR = BUCK2 = 1V1 ( cont. 1000mA) (Ind. Peak 1.6A)\nVDD = BUCK3 = 3V3 (cont. 500mA) (Ind. Peak 1A)\nUNUSED = BUCK 4 = 1V2 (cont. 2000mA) (Ind. Peak 3A)\nSWITCHING FREQ: 2MHz\nDigi P/N for inductors for dev board bucks: 490-10647-1-ND"
- note removed: "VDD_CORE = BUCK1 = 1V2\nVDD_DDR = BUCK2 = 1V1\nVDD = BUCK3 = 3V3\n"
- moved on the sheet: C?, L?, R?, SW?, U?
