File: stm32mpu/stm32mpu/stm32mpu.sch (KiCad schematic (older format))
At the start: 0 parts

Commit message: pre-leaving newfoundland
added a lot of stuff - unsure of what has changed
Other:
- note added: "- 100Base-TX Ethernet\n- SD Card boot storage"
- note added: "- SD Card boot medium\n- 1 Gbit DDR3L RAM"
- note added: "Breakout board for the STM32MP157AAA3T MPU from ST Microelectronics\n"
- note added: "Digikey P/N for MPU: 497-19096-1-ND\nDigikey P/N for PMIC: 497-19781-1-ND\nDigikey P/N for DRAM: 557-2010-1-ND\nDigikey P/N for Ethernet PHY: 296-39561-1-ND"
- note added: "ETHERNET"
- note added: "FLASH (SD) &\nCORE MISC."
- note added: "PERIPHERAL\nBREAKOUT"
- note added: "STM32MP157A BREAKOUT BOARD"
- note removed: "Digikey P/N for MPU: 497-19096-1-ND\nDigikey P/N for PMIC: 497-19781-1-ND\nDigikey P/N for DRAM: 557-2010-1-ND\nDigikey P/N for Ethernet PHY: 576-4177-1-ND"
- note removed: "FLASH +\nETHERNET"
Changed lines of the file:
@@
 $Descr A4 11693 8268
 encoding utf-8
-Sheet 1 4
+Sheet 1 7
 Title ""
 Date ""
@@
 Comment4 ""
 $EndDescr
-Text Notes 4750 1050 0    50   ~ 0
-Digikey P/N for MPU: 497-19096-1-ND\nDigikey P/N for PMIC: 497-19781-1-ND\nDigikey P/N for DRAM: 557-2010-1-ND\nDigikey P/N for Ethernet PHY: 576-4177-1-ND
+Text Notes 4550 7600 0    50   ~ 0
+Digikey P/N for MPU: 497-19096-1-ND\nDigikey P/N for PMIC: 497-19781-1-ND\nDigikey P/N for DRAM: 557-2010-1-ND\nDigikey P/N for Ethernet PHY: 296-39561-1-ND
 $Sheet
-S 1800 1950 2550 1300
+S 1750 2700 2550 1300
 U 607DAB58
 F0 "power" 50
@@
 $EndSheet
 $Sheet
-S 7750 2000 2550 1300
+S 4900 2700 2550 1300
 U 607DAC09
 F0 "RAM" 50
@@
 $EndSheet
 $Sheet
-S 4700 4100 2550 1300
+S 1650 4750 2550 1300
 U 607DAC6D
-F0 "peripherals" 50
-F1 "peripherals.sch" 50
+F0 "ethernet" 50
+F1 "ethernet.sch" 50
 $EndSheet
-Text Notes 2700 2700 0    118  ~ 24
+Text Notes 2650 3450 0    118  ~ 24
 POWER
-Text Notes 8700 2750 0    118  ~ 24
+Text Notes 5850 3450 0    118  ~ 24
 MEMORY
-Text Notes 5500 4950 0    118  ~ 24
-FLASH +\nETHERNET
+Text Notes 2400 5500 0    118  ~ 24
+ETHERNET
+$Sheet
+S 4900 4700 2550 1300
+U 611188A5
+F0 "Flash" 50
+F1 "Flash.sch" 50
+$EndSheet
+Text Notes 5600 5500 0    118  ~ 24
+FLASH (SD) &\nCORE MISC.
+Text Notes 3650 1550 0    197  ~ 39
+STM32MP157A BREAKOUT BOARD
+Text Notes 3850 1750 0    79   Italic 0
+Breakout board for the STM32MP157AAA3T MPU from ST Microelectronics\n
+Text Notes 8700 4600 0    118  ~ 24
+PERIPHERAL\nBREAKOUT
+$Sheet
+S 8000 3750 2550 1300
+U 60F3B124
+F0 "preph_breakout" 50
+F1 "preph_breakout.sch" 50
+$EndSheet
+Text Notes 4550 2000 0    59   ~ 0
+- SD Card boot medium\n- 1 Gbit DDR3L RAM
+Text Notes 6100 2000 0    59   ~ 0
+- 100Base-TX Ethernet\n- SD Card boot storage
 $EndSCHEMATC
